Commit message: Traquad: wheel_rad 0.045, tracks up to 1 m/s, IK model fitted with the Qualisys
- wheel_rad 0.045 (Qualisys: base speed / joint speed on straight runs, 0.0454 m)
- track joints max_velocity 25 rad/s (legs stay at 10) and twist_max_x 1.0 m/s
- TraquadIK: effective half track y0 − kδ·|δ| from the yaw posture of the hips
  (δ = mean HFE angle), forward creep d·|ωz| while turning, optional compensation
  of the track deficit (Kd-only drives), replacing γ·X̄; tests updated
- identify_yaw_slip.py removed (it identified γ); analysis scripts at r 0.045

Claude-Session: https://claude.ai/code/session_01DPhTMkZzZXespjTiHcSZRs

File: src/pi3hat/pi3hat_hw_interface/urdf/traquad8_dji.xacro (robot description, xacro)
@@ -1,5 +1,5 @@
 <?xml version="1.0" ?>
 <robot name="omnicar"  xmlns:xacro="http://ros.org/wiki/xacro">
-    <xacro:macro name="joint" params="name id bus kp kd second_encoder_source max_pos_limit min_pos_limit actuator_trasmission max_current_A">
+    <xacro:macro name="joint" params="name id bus kp kd second_encoder_source max_pos_limit min_pos_limit actuator_trasmission max_current_A max_velocity">
         <joint name="${name}">
             <param name="id">${id}</param>
@@ -17,5 +17,5 @@
             <param name="max_pos_limit">${max_pos_limit}</param>
             <param name="min_pos_limit">${min_pos_limit}</param>
-            <param name="max_velocity">10.0</param>
+            <param name="max_velocity">${max_velocity}</param>
             <param name="max_effort">15.0</param>
             <param name="actuator_trasmission">${actuator_trasmission}</param>
@@ -43,8 +43,10 @@
     </xacro:macro>
      <xacro:macro name="leg_joint" params="name id bus">
-     <xacro:joint name="${name}" id="${id}" bus="${bus}" kp="60.0" kd="0.6" second_encoder_source="-1" max_pos_limit="3.14" min_pos_limit="-3.14" actuator_trasmission="9" max_current_A="80.0"/>
+     <xacro:joint name="${name}" id="${id}" bus="${bus}" kp="60.0" kd="0.6" second_encoder_source="-1" max_pos_limit="3.14" min_pos_limit="-3.14" actuator_trasmission="9" max_current_A="80.0" max_velocity="10.0"/>
     </xacro:macro>
+    <!-- Track joints: max_velocity 25 rad/s (1.1 m/s with wheel_rad 0.045; was 10 as the legs, about 0.45 m/s).
+         The moteus derate the torque above it, so the tracks can still go about 1.5 rad/s past it -->
     <xacro:macro name="wheel_joint" params="name id bus">
-        <xacro:joint name="${name}" id="${id}" bus="${bus}" kp="0.0" kd="0.9" second_encoder_source="-1" max_pos_limit="5000.0" min_pos_limit="-5000.0" actuator_trasmission="15" max_current_A="40.0"/>
+        <xacro:joint name="${name}" id="${id}" bus="${bus}" kp="0.0" kd="0.9" second_encoder_source="-1" max_pos_limit="5000.0" min_pos_limit="-5000.0" actuator_trasmission="15" max_current_A="40.0" max_velocity="25.0"/>
     </xacro:macro>
     <xacro:macro name="distributor_joint" params="name id">
